Commit message: Finally a goddamn robot that moves without looking like a retard!

File: assing2/catkin_ws/src/reactive_bot_description/urdf/reactive_bot.xacro (robot description, xacro)
@@ -1,84 +1,323 @@
 <?xml version="1.0" ?>
-<robot name="reactive_bot" xmlns:xacro="http://www.ros.org/wiki/xacro" >
-  <xacro:include filename="$(find reactive_bot_description)/urdf/materials.xacro" />
-  <xacro:include filename="$(find reactive_bot_description)/urdf/gazebo.xacro" />
-  <xacro:include filename="$(find reactive_bot_description)/urdf/macro.xacro" />
-  <link name="link_chassis">
-    <!-- pose and inertial -->
-    <pose>0 0 0.1 0 0 0</pose>
+<robot name="reactive_bot"
+  xmlns:xacro="http://www.ros.org/wiki/xacro">
+  <!-- Based on this: https://github.com/qboticslabs/mastering_ros/blob/master/chapter_2_codes/mastering_ros_robot_description_pkg/urdf/diff_wheeled_robot.xacro -->
+  <!-- Wheels -->
+  <!-- in kg-->
+  <!-- Defining the colors used in this robot -->
+  <material name="Black">
+    <color rgba="0.0 0.0 0.0 1.0"/>
+  </material>
+  <material name="White">
+    <color rgba="1.0 1.0 1.0 1.0"/>
+  </material>
+  <material name="Blue">
+    <color rgba="0.0 0.0 0.8 1.0"/>
+  </material>
+  <!-- PROPERTY LIST -->
+  <!--All units in m-kg-s-radians unit system -->
+  <!-- Main body radius and height -->
+  <!-- Main Body Cylinder base   -->
+  <!-- in kg-->
+  <!-- caster wheel radius and height -->
+  <!-- caster wheel mass -->
+  <!-- in kg-->
+  <!-- caster wheel radius and height -->
+  <!-- caster wheel mass -->
+  <!-- in kg-->
+  <!-- Wheels -->
+  <!-- in kg-->
+  <!-- Hokuyo Laser scanner -->
+  <!-- Macro for calculating inertia of cylinder -->
+  <!-- BASE-FOOTPRINT -->
+  <!-- link_base_footprint is a fictitious link(frame) that is on the ground right below link_base origin -->
+  <link name="link_base_footprint">
+    <inertial>
+      <mass value="0.0001"/>
+      <origin xyz="0 0 0"/>
+      <inertia ixx="0.0001" ixy="0.0" ixz="0.0" iyy="0.0001" iyz="0.0" izz="0.0001"/>
+    </inertial>
+    <visual>
+      <origin rpy="0 0 0" xyz="0 0 0"/>
+      <geometry>
+        <box size="0.001 0.001 0.001"/>
+      </geometry>
+    </visual>
+  </link>
+  <gazebo reference="link_base_footprint">
+    <turnGravityOff>false</turnGravityOff>
+  </gazebo>
+  <joint name="link_base_footprint_joint" type="fixed">
+    <origin rpy="0 0 0" xyz="0 0 0.04"/>
+    <parent link="link_base_footprint"/>
+    <child link="link_base"/>
+  </joint>
+  <!-- BASE-LINK -->
+  <!--Actual body/chassis of the robot-->
+  <link name="link_base">
     <inertial>
       <mass value="5"/>
-      <origin rpy="0 0 0" xyz="0 0 0.1"/>
-      <inertia ixx="0.0395416666667" ixy="0" ixz="0" iyy="0.106208333333" iyz="0" izz="0.106208333333"/>
-    </inertial>
-    <!-- body -->
-    <collision name="collision_chassis">
-      <geometry>
-        <box size="0.5 0.3 0.07"/>
-      </geometry>
-    </collision>
+      <origin xyz="0 0 0"/>
+      <!--The 3x3 rotational inertia matrix. -->
+      <inertia ixx="0.0282916666667" ixy="0" ixz="0" iyy="0.0282916666667" iyz="0" izz="0.05625"/>
+    </inertial>
     <visual>
       <origin rpy="0 0 0" xyz="0 0 0"/>
       <geometry>
-        <box size="0.5 0.3 0.07"/>
-      </geometry>
-      <material name="blue"/>
-    </visual>
-    <!-- caster front -->
-    <collision name="caster_front_collision">
-      <origin rpy=" 0 0 0" xyz="0.35 0 -0.05"/>
-      <geometry>
-        <sphere radius="0.05"/>
-      </geometry>
-      <surface>
-        <friction>
-          <ode>
-            <mu>0</mu>
-            <mu2>0</mu2>
-            <slip1>1.0</slip1>
-            <slip2>1.0</slip2>
-          </ode>
-        </friction>
-      </surface>
-    </collision>
-    <visual name="caster_front_visual">
-      <origin rpy=" 0 0 0" xyz="0.2 0 -0.05"/>
-      <geometry>
-        <sphere radius="0.05"/>
-      </geometry>
-    </visual>
-  </link>
-  <!-- Create wheel right -->
-  <xacro:link_wheel name="link_right_wheel" />
-  <!--   Joint for right wheel  -->
-  <xacro:joint_wheel name="joint_right_wheel" child="link_right_wheel" origin_xyz="-0.05 0.20 0" />
-  <!-- Left Wheel link -->
-  <xacro:link_wheel name="link_left_wheel" />
-  <!--   Joint for left wheel  -->
-  <xacro:joint_wheel name="joint_left_wheel" child="link_left_wheel" origin_xyz="-0.05 -0.20 0" />
-  <link name="sensor_laser">
-    <inertial>
-      <origin xyz="0 0 0" rpy="0 0 0" />
-      <mass value="1" />
-      <xacro:cylinder_inertia mass="1" r="0.05" l="0.1" />
-    </inertial>
-    <visual>
-      <origin xyz="0 0 0" rpy="0 0 0" />
-      <geometry>
-        <cylinder radius="0.05" length="0.1"/>
-      </geometry>
-      <material name="white" />
-    </visual>
-    <collision>
-      <origin xyz="0 0 0" rpy="0 0 0"/>
-      <geometry>
-        <cylinder radius="0.05" length="0.1"/>
-      </geometry>
-    </collision>
-  </link>
-  <joint name="joint_sensor_laser" type="fixed">
-    <origin xyz="0.15 0 0.05" rpy="0 0 0"/>
-    <parent link="link_chassis"/>
-    <child link="sensor_laser"/>
-  </joint>
+        <cylinder length="0.02" radius="0.15"/>
+      </geometry>
+      <material name="White"/>
+    </visual>
+    <collision>
+      <origin rpy="0 0 0 " xyz="0 0 0"/>
+      <geometry>
+        <cylinder length="0.02" radius="0.15"/>
+      </geometry>
+    </collision>
+  </link>
+  <gazebo reference="link_base">
+    <material>Gazebo/White</material>
+    <turnGravityOff>false</turnGravityOff>
+  </gazebo>
+  <!-- RIGHT WHEEL -->
+  <link name="link_right_wheel">
+    <visual>
+      <origin rpy="1.57079632679 0  0 " xyz="0 0 0"/>
+      <geometry>
+        <cylinder length="0.02" radius="0.04"/>
+      </geometry>
+      <material name="DarkGray"/>
+    </visual>
+    <collision>
+      <origin rpy="1.57079632679 0 0 " xyz="0 0 0"/>
+      <geometry>
+        <cylinder length="0.02" radius="0.04"/>
+      </geometry>
+    </collision>
+    <inertial>
+      <mass value="2.5"/>
+      <origin xyz="0 0 0"/>
+      <inertia ixx="0.00108333333333" ixy="0" ixz="0" iyy="0.00108333333333" iyz="0" izz="0.002"/>
+    </inertial>
+  </link>
+  <gazebo reference="link_right_wheel">
+    <mu1 value="1.0"/>
+    <mu2 value="1.0"/>
+    <kp value="10000000.0"/>
+    <kd value="1.0"/>
+    <fdir1 value="1 0 0"/>
+    <material>Gazebo/Grey</material>
+    <turnGravityOff>false</turnGravityOff>
+  </gazebo>
+  <joint name="joint_right_wheel" type="continuous">
+    <parent link="link_base"/>
+    <child link="link_right_wheel"/>
+    <origin rpy="0 0 0" xyz="0.0 0.15 0.0"/>
+    <axis rpy="0  0" xyz="0 1 0"/>
+    <limit effort="100" velocity="100"/>
+    <joint_properties damping="0.0" friction="0.0"/>
+  </joint>
+  <!-- Transmission is important to link the joints and the controller -->
+  <transmission name="joint_right_wheel_trans">
+    <type>transmission_interface/SimpleTransmission</type>
+    <joint name="joint_right_wheel"/>
+    <actuator name="joint_right_wheel_motor">
+      <hardwareInterface>EffortJointInterface</hardwareInterface>
+      <mechanicalReduction>1</mechanicalReduction>
+    </actuator>
+  </transmission>
+  <!--LEFT WHEEL -->
+  <link name="link_left_wheel">
+    <visual>
+      <origin rpy="1.57079632679 0  0 " xyz="0 0 0"/>
+      <geometry>
+        <cylinder length="0.02" radius="0.04"/>
+      </geometry>
+      <material name="DarkGray"/>
+    </visual>
+    <collision>
+      <origin rpy="1.57079632679 0 0 " xyz="0 0 0"/>
+      <geometry>
+        <cylinder length="0.02" radius="0.04"/>
+      </geometry>
+    </collision>
+    <inertial>
+      <mass value="2.5"/>
+      <origin xyz="0 0 0"/>
+      <inertia ixx="0.00108333333333" ixy="0" ixz="0" iyy="0.00108333333333" iyz="0" izz="0.002"/>
+    </inertial>
+  </link>
+  <gazebo reference="link_left_wheel">
+    <mu1 value="1.0"/>
+    <mu2 value="1.0"/>
+    <kp value="10000000.0"/>
+    <kd value="1.0"/>
+    <fdir1 value="1 0 0"/>
+    <material>Gazebo/Grey</material>
+    <turnGravityOff>false</turnGravityOff>
+  </gazebo>
+  <joint name="joint_left_wheel" type="continuous">
+    <parent link="link_base"/>
+    <child link="link_left_wheel"/>
+    <origin rpy="0 0 0" xyz="0.0 -0.15 0.0"/>
+    <axis rpy="0  0" xyz="0 1 0"/>
+    <limit effort="100" velocity="100"/>
+    <joint_properties damping="0.0" friction="0.0"/>
+  </joint>
+  <!-- Transmission is important to link the joints and the controller -->
+  <transmission name="joint_left_wheel_trans">
+    <type>transmission_interface/SimpleTransmission</type>
+    <joint name="joint_left_wheel"/>
+    <actuator name="joint_left_wheel_motor">
+      <hardwareInterface>EffortJointInterface</hardwareInterface>
+      <mechanicalReduction>1</mechanicalReduction>
+    </actuator>
+  </transmission>
+  <!-- FRONT CASTER  -->
+  <link name="link_front_caster">
+    <visual>
+      <origin rpy="1.57079632679 0 0" xyz="0 0.02 0"/>
+      <geometry>
+        <sphere radius="0.025"/>
+      </geometry>
+      <material name="Black"/>
+    </visual>
+    <collision>
+      <geometry>
+        <sphere radius="0.025"/>
+      </geometry>
+      <origin rpy="1.57079632679 0 0" xyz="0 0.02 0"/>
+    </collision>
+    <inertial>
+      <mass value="0.5"/>
+      <origin xyz="0 0 0"/>
+      <inertia ixx="0.001" ixy="0.0" ixz="0.0" iyy="0.001" iyz="0.0" izz="0.001"/>
+    </inertial>
+  </link>
+  <joint name="caster_front_joint" type="fixed">
+    <parent link="link_base"/>
+    <child link="link_front_caster"/>
+    <origin rpy="-1.57079632679 0 0" xyz="0.115 0.0 0.007"/>
+  </joint>
+  <gazebo reference="link_front_caster">
+    <turnGravityOff>false</turnGravityOff>
+  </gazebo>
+  <!--BACK CASTER  -->
+  <link name="link_back_caster">
+    <visual>
+      <origin rpy="1.57079632679 0 0" xyz="0.02 0.02 0 "/>
+      <geometry>
+        <sphere radius="0.025"/>
+      </geometry>
+      <material name="Black"/>
+    </visual>
+    <collision>
+      <geometry>
+        <sphere radius="0.025"/>
+      </geometry>
+      <origin rpy="1.57079632679 0 0" xyz="0 0.02 0 "/>
+    </collision>
+    <inertial>
+      <mass value="0.5"/>
+      <origin xyz="0 0 0"/>
+      <inertia ixx="0.001" ixy="0.0" ixz="0.0" iyy="0.001" iyz="0.0" izz="0.001"/>
+    </inertial>
+  </link>
+  <joint name="caster_back_joint" type="fixed">
+    <parent link="link_base"/>
+    <child link="link_back_caster"/>
+    <origin rpy="-1.57079632679 0 0" xyz="-0.135 0.0 0.009"/>
+  </joint>
+  <gazebo reference="link_back_caster">
+    <turnGravityOff>false</turnGravityOff>
+  </gazebo>
+  <!-- SENSORS -->
+  <!-- LASER SCAN a.k.a. Hokuyo -->
+  <link name="link_hokuyo">
+    <visual>
+      <origin rpy="0 0 0" xyz="0 0 0"/>
+      <geometry>
+        <box size="0.05 0.05 0.1"/>
+      </geometry>
+      <material name="Blue"/>
+    </visual>
+  </link>
+  <joint name="joint_hukuyo" type="fixed">
+    <origin rpy="0 0 0" xyz="0.125 0 0.05"/>
+    <parent link="link_base"/>
+    <child link="link_hokuyo"/>
+  </joint>
+  <gazebo reference="link_hokuyo">
+    <material>Gazebo/Blue</material>
+    <turnGravityOff>false</turnGravityOff>
+    <sensor name="head_hokuyo_sensor" type="ray">
+      <pose>0.025 0 0 0 0 0</pose>
+      <visualize>true</visualize>
+      <update_rate>40</update_rate>
+      <ray>
+        <scan>
+          <horizontal>
+            <samples>720</samples>
+            <resolution>1</resolution>
+            <min_angle>-3.14</min_angle>
+            <max_angle>3.14</max_angle>
+          </horizontal>
+        </scan>
+        <range>
+          <min>0.10</min>
+          <max>10.0</max>
+          <resolution>0.001</resolution>
+        </range>
+      </ray>
+      <plugin filename="libgazebo_ros_laser.so" name="gazebo_ros_hokuyo_controller">
+        <topicName>/scan</topicName>
+        <frameName>link_hokuyo</frameName>
+      </plugin>
+    </sensor>
+  </gazebo>
+  <!-- Differential drive controller  -->
+  <!-- <gazebo>
+    <plugin filename="libgazebo_ros_diff_drive.so" name="differential_drive_controller_front">
+      <rosDebugLevel>Debug</rosDebugLevel>
+      <publishWheelTF>True</publishWheelTF>
+      <publishTf>1</publishTf>
+      <publishWheelJointState>true</publishWheelJointState>
+      <alwaysOn>true</alwaysOn>
+      <updateRate>100.0</updateRate>
+      <leftJoint>joint_left_wheel</leftJoint>
+      <rightJoint>joint_right_wheel</rightJoint>
+      <wheelSeparation>0.3</wheelSeparation>
+      <wheelDiameter>0.08</wheelDiameter>
+      <broadcastTF>1</broadcastTF>
+      <wheelTorque>30</wheelTorque>
+      <wheelAcceleration>1.8</wheelAcceleration>
+      <commandTopic>cmd_vel</commandTopic>
+      <odometryFrame>odom</odometryFrame>
+      <odometryTopic>odom</odometryTopic>
+      <robotBaseFrame>link_base</robotBaseFrame>
+    </plugin>
+  </gazebo> -->
+  <!--
+	  <gazebo>
+	    <plugin name="kobuki_controller" filename="libgazebo_ros_kobuki.so">
+	      <publish_tf>1</publish_tf>
+	      <left_wheel_joint_name>joint_left_wheel</left_wheel_joint_name>
+	      <right_wheel_joint_name>joint_right_wheel</right_wheel_joint_name>
+	      <wheel_separation>.30</wheel_separation>
+	      <wheel_diameter>0.08</wheel_diameter>
+	      <torque>30.0</torque>
+	      <velocity_command_timeout>0.6</velocity_command_timeout>
+	    </plugin>
+	  </gazebo>
+-->
+  <!--
+<gazebo>
+    <plugin name="gazebo_ros_control" filename="libgazebo_ros_control.so" />
+    <plugin filename="libgazebo_ros_joint_state_publisher.so" name="joint_state_publisher">
+      <jointName>joint_right_wheel, joint_left_wheel</jointName>
+      <updateRate>10.0</updateRate>
+      <alwaysOn>true</alwaysOn>
+    </plugin>
+</gazebo>
+-->
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
Commit message: differtential drive with keys working

File: assing2/catkin_ws/src/reactive_bot_description/urdf/reactive_bot.xacro (robot description, xacro)
@@ -65,5 +65,5 @@
       <origin rpy="0 0 0" xyz="0 0 0"/>
       <geometry>
-        <cylinder length="0.02" radius="0.15"/>
+        <cylinder length="0.02" radius="0.1"/>
       </geometry>
       <material name="White"/>
@@ -72,5 +72,5 @@
       <origin rpy="0 0 0 " xyz="0 0 0"/>
       <geometry>
-        <cylinder length="0.02" radius="0.15"/>
+        <cylinder length="0.02" radius="0.1"/>
       </geometry>
     </collision>
@@ -113,5 +113,5 @@
     <parent link="link_base"/>
     <child link="link_right_wheel"/>
-    <origin rpy="0 0 0" xyz="0.0 0.15 0.0"/>
+    <origin rpy="0 0 0" xyz="0.0 0.1 0.0"/>
     <axis rpy="0  0" xyz="0 1 0"/>
     <limit effort="100" velocity="100"/>
@@ -160,5 +160,5 @@
     <parent link="link_base"/>
     <child link="link_left_wheel"/>
-    <origin rpy="0 0 0" xyz="0.0 -0.15 0.0"/>
+    <origin rpy="0 0 0" xyz="0.0 -0.1 0.0"/>
     <axis rpy="0  0" xyz="0 1 0"/>
     <limit effort="100" velocity="100"/>
@@ -198,5 +198,5 @@
     <parent link="link_base"/>
     <child link="link_front_caster"/>
-    <origin rpy="-1.57079632679 0 0" xyz="0.115 0.0 0.007"/>
+    <origin rpy="-1.57079632679 0 0" xyz="0.075 0.0 0.007"/>
   </joint>
   <gazebo reference="link_front_caster">
@@ -227,5 +227,5 @@
     <parent link="link_base"/>
     <child link="link_back_caster"/>
-    <origin rpy="-1.57079632679 0 0" xyz="-0.135 0.0 0.009"/>
+    <origin rpy="-1.57079632679 0 0" xyz="-0.100 0.0 0.007"/>
   </joint>
   <gazebo reference="link_back_caster">
@@ -277,6 +277,6 @@
   </gazebo>
   <!-- Differential drive controller  -->
-  <!-- <gazebo>
-    <plugin filename="libgazebo_ros_diff_drive.so" name="differential_drive_controller_front">
+  <gazebo>
+    <plugin filename="libgazebo_ros_diff_drive.so" name="differential_drive_controller">
       <rosDebugLevel>Debug</rosDebugLevel>
       <publishWheelTF>True</publishWheelTF>
@@ -292,4 +292,7 @@
       <wheelTorque>30</wheelTorque>
       <wheelAcceleration>1.8</wheelAcceleration>
+      <!-- This defines the topic to which we should publish the message to control the bot. -->
+      <!-- In this plugin, the type of message is Twist (sensor_msgs/Twist). -->
+      <!-- Therefore the controller only needs to publish a Twist message to the /cmd_vel topic. -->
       <commandTopic>cmd_vel</commandTopic>
       <odometryFrame>odom</odometryFrame>
@@ -297,27 +300,4 @@
       <robotBaseFrame>link_base</robotBaseFrame>
     </plugin>
-  </gazebo> -->
-  <!--
-	  <gazebo>
-	    <plugin name="kobuki_controller" filename="libgazebo_ros_kobuki.so">
-	      <publish_tf>1</publish_tf>
-	      <left_wheel_joint_name>joint_left_wheel</left_wheel_joint_name>
-	      <right_wheel_joint_name>joint_right_wheel</right_wheel_joint_name>
-	      <wheel_separation>.30</wheel_separation>
-	      <wheel_diameter>0.08</wheel_diameter>
-	      <torque>30.0</torque>
-	      <velocity_command_timeout>0.6</velocity_command_timeout>
-	    </plugin>
-	  </gazebo>
--->
-  <!--
-<gazebo>
-    <plugin name="gazebo_ros_control" filename="libgazebo_ros_control.so" />
-    <plugin filename="libgazebo_ros_joint_state_publisher.so" name="joint_state_publisher">
-      <jointName>joint_right_wheel, joint_left_wheel</jointName>
-      <updateRate>10.0</updateRate>
-      <alwaysOn>true</alwaysOn>
-    </plugin>
-</gazebo>
--->
+  </gazebo>
 </robot>

Commit message: Fixed diff drive model deleting problem

File: assing2/catkin_ws/src/reactive_bot_description/urdf/reactive_bot.xacro (robot description, xacro)
@@ -244,5 +244,5 @@
   </link>
   <joint name="joint_hukuyo" type="fixed">
-    <origin rpy="0 0 0" xyz="0.125 0 0.05"/>
+    <origin rpy="0 0 0" xyz="0.075 0 0.05"/>
     <parent link="link_base"/>
     <child link="link_hokuyo"/>
@@ -251,12 +251,13 @@
     <material>Gazebo/Blue</material>
     <turnGravityOff>false</turnGravityOff>
+    <!-- Reference: http://wiki.ros.org/urdf/XML/sensor and http://sdformat.org/spec?ver=1.6&elem=sensor-->
     <sensor name="head_hokuyo_sensor" type="ray">
       <pose>0.025 0 0 0 0 0</pose>
       <visualize>true</visualize>
-      <update_rate>40</update_rate>
+      <update_rate>20</update_rate>
       <ray>
         <scan>
           <horizontal>
-            <samples>720</samples>
+            <samples>1080</samples>
             <resolution>1</resolution>
             <min_angle>-3.14</min_angle>
@@ -271,5 +272,5 @@
       </ray>
       <plugin filename="libgazebo_ros_laser.so" name="gazebo_ros_hokuyo_controller">
-        <topicName>/scan</topicName>
+        <topicName>/reactive_bot/laser/scan</topicName>
         <frameName>link_hokuyo</frameName>
       </plugin>
@@ -278,5 +279,8 @@
   <!-- Differential drive controller  -->
   <gazebo>
-    <plugin filename="libgazebo_ros_diff_drive.so" name="differential_drive_controller">
+    <!-- Issue with this plugin when deleting model in Gazebo: https://github.com/ros-simulation/gazebo_ros_pkgs/issues/123 -->
+    <!-- Therefore I created my own plugin in my_diff_drive package -->
+    <!-- <plugin filename="libgazebo_ros_diff_drive.so" name="differential_drive_controller"> -->
+    <plugin filename="my_ros_diff_drive.so" name="my_diff_drive">
       <rosDebugLevel>Debug</rosDebugLevel>
       <publishWheelTF>True</publishWheelTF>

Commit message: Changed sensor angle because of Gazebo bug.

File: assing2/catkin_ws/src/reactive_bot_description/urdf/reactive_bot.xacro (robot description, xacro)
@@ -238,5 +238,5 @@
       <origin rpy="0 0 0" xyz="0 0 0"/>
       <geometry>
-        <box size="0.05 0.05 0.1"/>
+        <box size="0.025 0.025 0.2"/>
       </geometry>
       <material name="Blue"/>
@@ -244,5 +244,5 @@
   </link>
   <joint name="joint_hukuyo" type="fixed">
-    <origin rpy="0 0 0" xyz="0.075 0 0.05"/>
+    <origin rpy="0 0 0" xyz="0.050 0 0.1"/>
     <parent link="link_base"/>
     <child link="link_hokuyo"/>
@@ -261,6 +261,6 @@
             <samples>1080</samples>
             <resolution>1</resolution>
-            <min_angle>-3.14</min_angle>
-            <max_angle>3.14</max_angle>
+            <min_angle>-1.57</min_angle>
+            <max_angle>+1.57</max_angle>
           </horizontal>
         </scan>
@@ -268,6 +268,11 @@
           <min>0.10</min>
           <max>10.0</max>
-          <resolution>0.001</resolution>
+          <resolution>0.01</resolution>
         </range>
+        <noise>
+          <type>gaussian</type>
+          <mean>0.0</mean>
+          <stddev>0.01</stddev>
+        </noise>
       </ray>
       <plugin filename="libgazebo_ros_laser.so" name="gazebo_ros_hokuyo_controller">

Commit message: Follows walls good!

File: assing2/catkin_ws/src/reactive_bot_description/urdf/reactive_bot.xacro (robot description, xacro)
@@ -113,5 +113,5 @@
     <parent link="link_base"/>
     <child link="link_right_wheel"/>
-    <origin rpy="0 0 0" xyz="0.0 0.1 0.0"/>
+    <origin rpy="0 0 0" xyz="0.0 -0.1 0.0"/>
     <axis rpy="0  0" xyz="0 1 0"/>
     <limit effort="100" velocity="100"/>
@@ -160,5 +160,5 @@
     <parent link="link_base"/>
     <child link="link_left_wheel"/>
-    <origin rpy="0 0 0" xyz="0.0 -0.1 0.0"/>
+    <origin rpy="0 0 0" xyz="0.0 0.1 0.0"/>
     <axis rpy="0  0" xyz="0 1 0"/>
     <limit effort="100" velocity="100"/>
